File: hardware/mini_game.kicad_sch (KiCad schematic)
At the start: 18 parts, among them Q1 MMBT3904LT1G, SW2 SW_Push, SW3 SW_Push, SW4 SW_Push, SW5 SW_Push, U1 XIAO-ESP32-C6-SMD, U2 ER_OLEDM0.91_1x-I2C, U3 ER_OLEDM0.91_1x-I2C

Commit message: all peripherals working
Parts:
- removed S2: Joystick_Generic, digikey-footprints:Switch_Nav_12.4x12.4mm_SMD_JS5208, symbol Mini_Game:Joystick_Generic
- added SW7, SW8, SW9: SW_Push, symbol Switch:SW_Push
Connections:
- net GNDREF: now also SW7.2, SW8.2, SW9.2
- net at U1.1 (D0): now also SW7.1
- net at U1.2 (D1): now also SW8.1
- net at U1.7 (D6): now also SW9.1
- no-connect marks 11 -> 9
